File: pcb/thermometer.kicad_pcb (KiCad board)
At the start: 2 copper layers, 39.4 x 24.8 mm, 18 parts, among them J1 USB_B_Micro, U1 ESP-01v090, U2 GY-87, U3 LM1117-3.3

Commit message: Update PCB
Connections:
- net Net-(R5-Pad2) renamed /SCL
- net Net-(R6-Pad2) renamed /SDA
