File: pcb/thermometer.sch (KiCad schematic (older format))
At the start: 18 parts, among them J1 USB_B_Micro, U1 ESP-01v090, U2 GY-87, U3 LM1117-3.3

Commit message: Update PCB
Connections:
- net SCL: now reaches R5.2, U2.3 (SCL)
- net SDA: now reaches R6.2, U2.4 (SDA)
Changed lines of the file:
@@
 Wire Wire Line
 	6300 1850 6300 2100
+Text Label 7750 5250 0    50   ~ 0
+SDA
+Text Label 7750 5050 0    50   ~ 0
+SCL
 $EndSCHEMATC
